File: schematics/pantry_signal_system/full_schema.sch (EAGLE design)
At the start: 80 parts, among them J1 JST-XH254-2P, J2 JST-XH254-3P, J3 JST-XH254-2P, J4 JST-XH254-3P, J5 JST-XH254-2P, J6 JST-XH254-2P, J7 JST-XH254-2P, J8 JST-XH254-2P, J9 USBASP_PIN, Q1 FDS4935A, Q12 STP14NM50N, Q13 STP14NM50N, Q14 2N3904, Q7 2N3904, Q8 2N3904, Q9 STP14NM50N, SW1 SWITCH, SW2 SWITCH, U1 MCP1703T-5002E/CB, U10 FAN73611, U11 FAN73611, U12 NC7WZ04, U2 AD8544, U3 ATTINY13, U4 ATMEGA328P, U5 MCP1703T-5002E/CB, U6 2004A I2C, U7 BME280BME280-CONNECTOR-ONLY, U8 E220-900T22D, U9 FAN73611

Commit message: Continue working under supply schematics and supply controller firmware
Parts:
- removed D9: MBR130LSFT1G, my_devices:D
- removed Q14, Q7: 2N3904, my_devices:TRANSISTOR_NPN
- added Q2, Q3: (no value), my_devices:TRANSISTOR_NPN
- added Q4, Q5: (no value), my_devices:TRANSISTOR_PNP
- added R12, R25, R27, R28: 1M, my_devices:R
- added R26: 2M, my_devices:R
- R21: value R -> 3K
Connections:
- removed net N$27: D9.P$1, Q14.E
- removed net N$5: Q7.B, R21.P$1
- removed net REQUEST_SUPPLY_MEASURE: J1.PIN1, J7.PIN2, R21.P$2, U4.PB2
- new net IS_ENABLE_RESERVE_+5V_INV: R22.P$1, U2.C_OUT
- new net N$17: Q2.B, R12.P$2
- new net N$25: Q3.B, R25.P$2
- new net N$30: J9.MISO, U3.PB1
- new net N$31: Q2.C, R26.P$1
- new net N$32: Q3.C, R27.P$1
- new net N$33: J9.RESET, R26.P$2, R27.P$2, R28.P$2, U3.PB5
- new net REQUEST_SUPPLY_MEASURE_INV: J1.PIN1, J7.PIN2, R21.P$1, U4.PB2
- new net SUPPLY_AVR_+5V: C4.P$1, J9.VCC, Q4.C, R28.P$1, U3.VCC
- net +5V: now also Q4.E; no longer Q7.C
- net GND: now also Q2.E, Q3.E
- net IS_12V_POWER_OK: now also U2.C+; no longer U2.C-
- net IS_ENABLE_RESERVE_+5V: now also R25.P$1; no longer J9.MISO, R22.P$1, U2.C_OUT, U3.PB1
- net IS_USE_RESERVE_BATTERY: now also R12.P$1; no longer U3.PB4
- net N$2: now also Q4.B, R21.P$2; no longer C4.P$1, J9.VCC, Q7.E, U3.VCC
- net N$26: now also Q5.C; no longer D9.P$2
- net N$28: now also Q5.B; no longer Q14.B
- net PRIMARY_VOLTAGE_LEVEL: now also U3.PB3; no longer J9.RESET, U3.PB5
- net RESERVE_+5V_SUPPLY: now also Q5.E; no longer Q14.C
- net RESERVE_VOLTAGE_LEVEL: now also U3.PB4; no longer U3.PB3
- net SUPPLY_CONTROL_+5V: now also U2.C-; no longer U2.C+
Other:
- moved on the sheet: BAT1, BAT2, BAT3, C1, C4, D1, D2, D7, FU1, FU2, FU3, J9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

Commit message: working under supply schematics. I think I solved problem with 'current battery in use' signal reading
Parts:
- removed Q8: 2N3904, my_devices:TRANSISTOR_NPN
- removed Q9: STP14NM50N, my_devices:MOSFET_N
- removed R27, R28: 1M, my_devices:R
- added D6, D9: MBR130LSFT1G, my_devices:D
- D5: value D -> MBR130LSFT1G
- FU3: value FU -> H520PT
- J1: value JST-XH254-2P -> USBASP_PIN; device my_devices:JST-XH254-2P -> my_devices:USBASP_PIN
- J4: value JST-XH254-3P -> JST-XH254-2P; device my_devices:JST-XH254-3P -> my_devices:JST-XH254-2P
- J5: value JST-XH254-2P -> JST-XH254-3P; device my_devices:JST-XH254-2P -> my_devices:JST-XH254-3P
- J9: value USBASP_PIN -> JST-XH254-2P; device my_devices:USBASP_PIN -> my_devices:JST-XH254-2P
- Q2, Q3: value (none) -> 2N3906BU; device my_devices:TRANSISTOR_NPN -> my_devices:TRANSISTOR_PNP
- Q4: value (none) -> STP14NM50N; device my_devices:TRANSISTOR_PNP -> my_devices:MOSFET_N
- Q5: value (none) -> 2N3904; device my_devices:TRANSISTOR_PNP -> my_devices:TRANSISTOR_NPN
- R10, R11, R15, R26: value 2M -> 1M
- R13: value GL5528 -> 1M; device my_devices:RF -> my_devices:R
- R16: value 2M -> 3K
- R17: value R -> 10K
- R18: value 2M -> 10K
- R19, R25: value 1M -> 620
- R20: value 620 -> 1M
- R21: value 3K -> 2M
- R22: value 1K -> 2M
- R24: value 1M -> GL5528; device my_devices:R -> my_devices:RF
- R4: value 1M -> 2M
- R5: device my_devices:R -> my_devices:RD3296-Z
- R6: value 1M -> 1K
- R7: device my_devices:RD3296-Z -> my_devices:R
- R8: value R -> 2M
- R9: value 620 -> 2M
- U1: value MCP1703T-5002E/CB -> NC7WZ04; device my_devices:VOLTAGE_REGULATOR -> my_devices:INVERTER._X2
- U10: value FAN73611 -> E220-900T22D; device my_devices:FAN73611 -> my_devices:LORA
- U11: value FAN73611 -> BME280BME280-CONNECTOR-ONLY; device my_devices:FAN73611 -> my_devices:BME280BME280-CONNECTOR-ONLY
- U12: value NC7WZ04 -> 2004A I2C; device my_devices:INVERTER._X2 -> my_devices:I2C_DISPLAY
- U3: value ATTINY13 -> FAN73611; device my_devices:ATTINY13 -> my_devices:FAN73611
- U4: value ATMEGA328P -> FAN73611; device my_devices:ATMEGA328P -> my_devices:FAN73611
- U6: value 2004A I2C -> MCP1703T-5002E/CB; device my_devices:I2C_DISPLAY -> my_devices:VOLTAGE_REGULATOR
- U7: value BME280BME280-CONNECTOR-ONLY -> ATTINY13; device my_devices:BME280BME280-CONNECTOR-ONLY -> my_devices:ATTINY13
- U8: value E220-900T22D -> FAN73611; device my_devices:LORA -> my_devices:FAN73611
- U9: value FAN73611 -> ATMEGA328P; device my_devices:FAN73611 -> my_devices:ATMEGA328P
- renumbered Q12 to Q7, Q13 to Q6
Connections:
- removed net N$17: Q2.B, R12.P$2
- removed net N$25: Q3.B, R25.P$2
- removed net N$30: J9.MISO, U3.PB1
- removed net N$31: Q2.C, R26.P$1
- removed net N$32: Q3.C, R27.P$1
- removed net N$33: J9.RESET, R26.P$2, R27.P$2, R28.P$2, U3.PB5
- new net N$27: D8.P$2, J1.RESET, R10.P$1, R11.P$2, U7.PB5
- new net N$5: D9.P$2, J1.MISO, R15.P$2, U7.PB1
- net +12V: now also C1.PIN_PLUS, D1.P$2, D2.P$2, D7.P$1, J2.PIN1, J5.PIN3, J7.PIN1, J9.PIN2, R5.P2, U8.VB, U8.VDD; no longer C2.PIN_PLUS, D3.P$2, D4.P$2, D8.P$1, J2.PIN3, J3.PIN1, J6.PIN1, J8.PIN2, R7.P2, U11.VB, U11.VDD
- net +5V: now also C2.PIN_PLUS, J5.PIN2, Q3.E, R20.P$1, R21.P$2, R22.P$2, R23.P$2, U10.VCC, U11.VCC, U12.VCC, U6.OUT, U9.AREF, U9.AVCC, U9.VCC; no longer C3.PIN_PLUS, J4.PIN2, Q4.E, R14.P$1, R15.P$2, R16.P$2, R8.P$2, U4.AREF, U4.AVCC, U4.VCC, U5.OUT, U6.VCC, U7.VCC, U8.VCC
- net ENABLE_DISPLAY: now also R19.P$1, U9.PC3; no longer R9.P$1, U4.PC3
- net ENABLE_DR\YER: now also U8.IN, U9.PB1; no longer U11.IN, U4.PB1
- net FLOODING_ALARM_INDOOR: now also FS2.P$1, R23.P$1, U9.PC0; no longer FS1.P$1, R15.P$1, U4.PC0
- net FLOODING_ALARM_OUTDOOR: now also FS1.P$1, R21.P$1, U9.PC1; no longer FS2.P$1, R16.P$1, U4.PC1
- net GND: now also J1.GND, J1.GND1, J2.PIN3, J4.PIN2, J5.PIN1, J9.PIN1, Q4.S, Q5.E, R11.P$1, R12.P$1, R13.P$1, R14.P$1, R15.P$1, R24.P$2, R26.P$1, R5.P1, U3.VS, U4.VS, U6.GND, U8.VS, U9.GND1; no longer J2.PIN1, J4.PIN3, J6.PIN2, J8.PIN1, J9.GND, J9.GND1, Q2.E, Q3.E, Q8.E, Q9.S, R13.P$2, R19.P$1, R24.P$1, R4.P$1, R6.P$1, R7.P1, U10.VS, U11.VS, U12.GND, U4.GND1, U9.VS
- net I2C_SCL: now also U11.SCL, U12.SCL, U9.PC4; no longer U4.PC4, U6.SCL, U7.SCL
- net I2C_SDA: now also U11.SDA, U12.SDA, U9.PC5; no longer U4.PC5, U6.SDA, U7.SDA
- net IS_12V_POWER_OK: now also R5.P3; no longer R7.P3
- net IS_ENABLE_RESERVE_+5V: now also D9.P$1; no longer R25.P$1
- net IS_ENABLE_RESERVE_+5V_INV: now also R6.P$1; no longer R22.P$1
- net IS_PRIMARY_BATTERY_OK: now also R3.P$2, U1.A1; no longer R10.P$2, U12.A1
- net IS_RESERVE_BATTERY_OK: now also D6.P$1, R4.P$1; no longer D5.P$1, R11.P$1
- net IS_USE_RESERVE_BATTERY: now also D8.P$1, U1.A2; no longer R12.P$1, U12.A2
- net LIGHT_SENSOR: now also R20.P$2, R24.P$1, U9.PC2; no longer R13.P$1, R14.P$2, U4.PC2
- net LORA_AUX: now also U10.AUX, U9.PD6; no longer U4.PD6, U8.AUX
- net LORA_M0M1: now also U10.M0, U10.M1, U9.PD7; no longer U4.PD7, U8.M0, U8.M1
- net LORA_RX: now also U10.RX, U9.PD4; no longer U4.PD4, U8.RX
- net LORA_TX: now also U10.TX, U9.PD3; no longer U4.PD3, U8.TX
- net N$1: now also D3.P$2, D4.P$2, D5.P$2, U5.IN; no longer D1.P$2, D2.P$2, D7.P$2, U1.IN
- net N$10: now also Q5.C, U12.GND; no longer Q8.C, U6.GND
- net N$11: now also Q5.B, R19.P$2; no longer Q8.B, R9.P$2
- net N$12: now also D1.P$1; no longer D3.P$1
- net N$13: now also D2.P$1; no longer D4.P$1
- net N$14: now also J8.PIN2; no longer J5.PIN2
- net N$15: now also J8.PIN1; no longer J5.PIN1
- net N$16: now also U9.PD2; no longer U4.PD2
- net N$18: now also U1.Y1, U3.IN; no longer U12.Y1, U9.IN
- net N$19: now also U1.Y2, U4.IN; no longer U10.IN, U12.Y2
- net N$2: now also Q3.B, R16.P$2; no longer Q4.B, R21.P$2
- net N$23: now also R25.P$1, R26.P$2; no longer R19.P$2, R20.P$1
- net N$24: now also R25.P$2; no longer R20.P$2
- net N$26: now also D7.P$2, Q2.C, U6.IN; no longer D8.P$2, Q5.C, U5.IN
- net N$28: now also Q2.B, R6.P$2; no longer Q5.B, R22.P$2
- net N$3: now also R3.P$1; no longer R10.P$1
- net N$4: now also J7.PIN2, Q4.D; no longer J3.PIN2, Q9.D
- net N$6: now also Q4.G, U8.HO; no longer Q9.G, U11.HO
- net N$7: now also R18.P$1, U9.PC6; no longer R8.P$1, U4.PC6
- net N$8: now also R4.P$2; no longer R11.P$2
- net N$9: now also D6.P$2; no longer D5.P$2
- net OPEN_DOOR_ALARM: now also R22.P$1, U9.PB3; no longer R18.P$1, U4.PB3
- net PRIMARY_SUPPLY_12V: now also D3.P$1, R8.P$2, U3.VB, U3.VDD; no longer D1.P$1, R3.P$2, U9.VB, U9.VDD
- net PRIMARY_VOLTAGE_LEVEL: now also R13.P$2, R8.P$1, U7.PB3; no longer R3.P$1, R4.P$2, U3.PB3
- net REQUEST_SUPPLY_MEASURE_INV: now also J3.PIN2, J6.PIN1, R16.P$1, U9.PB2; no longer J1.PIN1, J7.PIN2, R21.P$1, U4.PB2
- net RESERVE_+5V_LEVEL: now also J1.SCK, R12.P$2, R7.P$1, U7.PB2; no longer J9.SCK, R23.P$1, R24.P$2, U3.PB2
- net RESERVE_+5V_SUPPLY: now also D5.P$1, Q2.E, R7.P$2; no longer D7.P$1, Q5.E, R23.P$2
- net RESERVE_SUPPLY_12V: now also D4.P$1, R9.P$2, U4.VB, U4.VDD; no longer D2.P$1, R5.P$2, U10.VB, U10.VDD
- net RESERVE_VOLTAGE_LEVEL: now also R14.P$2, R9.P$1, U7.PB4; no longer R5.P$1, R6.P$2, U3.PB4
- net SUPPLY_AVR_+5V: now also J1.VCC, Q3.C, U7.VCC; no longer J9.VCC, Q4.C, R28.P$1, U3.VCC
- net SUPPLY_CONTROL_+5V: now also C3.PIN_PLUS, R10.P$2, U1.VCC, U5.OUT; no longer C1.PIN_PLUS, U1.OUT, U12.VCC
- net SUPPLY_UART_TX: now also J1.MOSI, J3.PIN1, J6.PIN2, U7.PB0, U9.PB0; no longer J1.PIN2, J7.PIN1, J9.MOSI, U3.PB0, U4.PB0
- net USE_PRIMARY_BATTERY: now also U3.HO; no longer U9.HO
- net USE_RESERVE_BATTERY: now also U4.HO; no longer U10.HO
Other:
- moved on the sheet: BAT1, BAT2, BAT3, C1, C2, C3, C4, D1, D2, D3, D4, D5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

Commit message: and another iteration for suplly avr data reading
Parts:
- removed D8, D9: MBR130LSFT1G, my_devices:D
- added C8: 10 uF, my_devices:C
- added Q8: FDS4935A, my_devices:MOSFET_P_X2
- added R27: 620, my_devices:R
- FU1, FU2, FU3: value H520PT -> H520PT / 0.5A
- R10: value 1M -> 3K
- R11, R15: value 1M -> 10K
Connections:
- removed net IS_ENABLE_RESERVE_+5V: D9.P$1
- removed net N$5: D9.P$2, J1.MISO, R15.P$2, U7.PB1
- new net CURRENT_SUPPLY_IN_USE: J1.MISO, R27.P$2, U7.PB1
- new net N$17: J1.RESET, U7.PB5
- new net N$25: Q8.S1, R10.P$1
- new net N$29: C8.PIN_PLUS, R10.P$2, R11.P$2, R15.P$2, R27.P$1
- net +5V: no longer Q3.E
- net GND: now also C8.PIN_GND, Q8.D11, Q8.D12, Q8.D21, Q8.D22; no longer R11.P$1
- net IS_ENABLE_RESERVE_+5V_INV: now also Q8.G2
- net IS_USE_RESERVE_BATTERY: now also Q8.G1; no longer D8.P$1
- net N$27: now also Q8.S2, R11.P$1; no longer D8.P$2, J1.RESET, R10.P$1, R11.P$2, U7.PB5
- net SUPPLY_CONTROL_+5V: now also Q3.E; no longer R10.P$2
Other:
- note added: "PRIMARY R = 10K & 10K = 5K RESERE R = 10K & 10K & 3K = 1.9K RESERVE 5V R = 10 K = 10K Time 5V to <3V: PRIMARY = 5K & 10 uF ~ 30 msec RESERVE = 1.9K & 10 uF ~ 10 msec RESERVE 5V = 10K & 10 uF ~ 60 msec"
- moved on the sheet: C4, J1, Q3, R10, R11, R12, R13, R14, R15, R16, R7, R8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

Commit message: Supply controller schematics and firmware ready
Parts:
- R10: value 3K -> 10K
- R11: value 10K -> 3K
Other:
- note added: "PRIMARY R = 10K & 10K = 5K RESERVE R = 10 K = 10K RESERE_5V R = 10K & 10K & 3K = 1.9K Time 5V to <3V (calculated): PRIMARY = 5K & 10 uF ~ 27 msec RESERVE = 10K & 10 uF ~ 60 msec RESERVE_5V = 1.9K & 10 uF ~ 10 msec Measured PRIMARY ~ 76 msec RESERVE ~ 114 msec RESERVE5V ~ 38 msec"
- note removed: "PRIMARY R = 10K & 10K = 5K RESERE R = 10K & 10K & 3K = 1.9K RESERVE 5V R = 10 K = 10K Time 5V to <3V: PRIMARY = 5K & 10 uF ~ 30 msec RESERVE = 1.9K & 10 uF ~ 10 msec RESERVE 5V = 10K & 10 uF ~ 60 msec"
- moved on the sheet: C4, C8, J1, Q3, R10, R11, R12, R13, R14, R15, R16, R27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

Commit message: working under supply schematics
Parts:
- removed Q8: FDS4935A, my_devices:MOSFET_P_X2
- removed R26: 1M, my_devices:R
- removed R27: 620, my_devices:R
- added D8: MBR130LSFT1G, my_devices:D
- added U13: 2004A I2C, my_devices:I2C_DISPLAY
- C4: value 0.1 uF -> 10 uF; device my_devices:C-1 -> my_devices:C
- C6: value 1000 uF -> 0.1 uF; device my_devices:C -> my_devices:C-1
- C8: value 10 uF -> 1000 uF
- Q2, Q3: value 2N3906BU -> FDS4935A; device my_devices:TRANSISTOR_PNP -> my_devices:MOSFET_P_X2
- R10: value 10K -> 2M
- R11, R16: value 3K -> 10K
- R15, R18: value 10K -> 620
- R19, R25: value 620 -> 1M
- R20: value 1M -> 2M
- R23: value 2M -> GL5528; device my_devices:R -> my_devices:RF
- R24: value GL5528 -> 620; device my_devices:RF -> my_devices:R
- R6: value 1K -> 10K
- R7: value 2M -> 3K
- U10: value E220-900T22D -> ATMEGA328P; device my_devices:LORA -> my_devices:ATMEGA328P
- U11: value BME280BME280-CONNECTOR-ONLY -> E220-900T22D; device my_devices:BME280BME280-CONNECTOR-ONLY -> my_devices:LORA
- U12: value 2004A I2C -> BME280BME280-CONNECTOR-ONLY; device my_devices:I2C_DISPLAY -> my_devices:BME280BME280-CONNECTOR-ONLY
- U7: value ATTINY13 -> FAN73611; device my_devices:ATTINY13 -> my_devices:FAN73611
- U8: value FAN73611 -> ATTINY13; device my_devices:FAN73611 -> my_devices:ATTINY13
- U9: value ATMEGA328P -> FAN73611; device my_devices:ATMEGA328P -> my_devices:FAN73611
Connections:
- removed net N$2: Q3.B, R16.P$2
- removed net N$28: Q2.B, R6.P$2
- new net N$5: D7.P$2, D8.P$2, U6.IN
- new net USE_RESERVE_5V_BATTERY: Q2.G2, U7.HO
- net +12V: now also U9.VB, U9.VDD; no longer U8.VB, U8.VDD
- net +5V: now also C3.PIN_PLUS, C7.PIN_PLUS, Q2.S1, R16.P$1, R17.P$2, R19.P$1, R20.P$2, U10.AREF, U10.AVCC, U13.VCC; no longer C2.PIN_PLUS, C6.PIN_PLUS, R17.P$1, R18.P$2, R20.P$1, R23.P$2, U9.AREF, U9.AVCC, U9.VCC
- net CURRENT_SUPPLY_IN_USE: now also R15.P$2, U8.PB1; no longer R27.P$2, U7.PB1
- net ENABLE_DISPLAY: now also R18.P$1, U10.PC3; no longer R19.P$1, U9.PC3
- net ENABLE_DR\YER: now also U10.PB1, U9.IN; no longer U8.IN, U9.PB1
- net FLOODING_ALARM_INDOOR: now also R22.P$1, U10.PC0; no longer R23.P$1, U9.PC0
- net FLOODING_ALARM_OUTDOOR: now also R20.P$1, U10.PC1; no longer R21.P$1, U9.PC1
- net GND: now also C4.PIN_GND, C6.P$2, Q3.D11, Q3.D12, Q3.D21, Q3.D22, R11.P$1, R23.P$2, R25.P$1, U10.GND1, U12.GND, U7.VS, U9.VS; no longer C4.P$2, C6.PIN_GND, Q8.D11, Q8.D12, Q8.D21, Q8.D22, R15.P$1, R24.P$2, R26.P$1, U8.VS, U9.GND1
- net I2C_SCL: now also U10.PC4, U13.SCL; no longer U11.SCL, U9.PC4
- net I2C_SDA: now also U10.PC5, U13.SDA; no longer U11.SDA, U9.PC5
- net IS_ENABLE_RESERVE_+5V_INV: now also Q3.G2, U7.IN; no longer Q8.G2, R6.P$1
- net IS_USE_RESERVE_BATTERY: now also Q3.G1; no longer Q8.G1
- net LIGHT_SENSOR: now also R19.P$2, R23.P$1, U10.PC2; no longer R20.P$2, R24.P$1, U9.PC2
- net LORA_AUX: now also U10.PD6, U11.AUX; no longer U10.AUX, U9.PD6
- net LORA_M0M1: now also U10.PD7, U11.M0, U11.M1; no longer U10.M0, U10.M1, U9.PD7
- net LORA_RX: now also U10.PD4, U11.RX; no longer U10.RX, U9.PD4
- net LORA_TX: now also U10.PD3, U11.TX; no longer U10.TX, U9.PD3
- net N$10: now also U13.GND; no longer U12.GND
- net N$11: now also R18.P$2; no longer R19.P$2
- net N$16: now also R16.P$2, U10.PD2; no longer R17.P$2, U9.PD2
- net N$17: now also U8.PB5; no longer U7.PB5
- net N$23: now also C8.PIN_PLUS, R24.P$1, R25.P$2; no longer C7.PIN_PLUS, R25.P$1, R26.P$2
- net N$24: now also R24.P$2; no longer R25.P$2
- net N$25: now also Q3.S1, R6.P$1; no longer Q8.S1, R10.P$1
- net N$26: now also D8.P$1, Q2.D21, Q2.D22; no longer D7.P$2, Q2.C, U6.IN
- net N$27: now also Q3.S2, R7.P$1; no longer Q8.S2, R11.P$1
- net N$29: now also C4.PIN_PLUS, R15.P$1, R6.P$2, R7.P$2; no longer C8.PIN_PLUS, R10.P$2, R15.P$2, R27.P$1
- net N$6: now also U9.HO; no longer U8.HO
- net N$7: now also C6.P$1, R17.P$1, U10.PC6; no longer C5.P$1, R18.P$1, U9.PC6
- net OPEN_DOOR_ALARM: now also R21.P$1, U10.PB3; no longer R22.P$1, U9.PB3
- net PRIMARY_SUPPLY_12V: now also R9.P$2; no longer R8.P$2
- net PRIMARY_VOLTAGE_LEVEL: now also R9.P$1, U8.PB3; no longer R8.P$1, U7.PB3
- net REQUEST_SUPPLY_MEASURE_INV: now also Q2.G1, U10.PB2; no longer R16.P$1, U9.PB2
- net RESERVE_+5V_LEVEL: now also R8.P$1, U8.PB2; no longer R7.P$1, U7.PB2
- net RESERVE_+5V_SUPPLY: now also Q2.S2, R8.P$2, U7.VB, U7.VDD; no longer Q2.E, R7.P$2
- net RESERVE_SUPPLY_12V: now also R10.P$2; no longer R9.P$2
- net RESERVE_VOLTAGE_LEVEL: now also R10.P$1, U8.PB4; no longer R9.P$1, U7.PB4
- net SUPPLY_AVR_+5V: now also C5.P$1, Q2.D11, Q2.D12, U8.VCC; no longer C4.P$1, Q3.C, U7.VCC
- net SUPPLY_CONTROL_+5V: now also C2.PIN_PLUS; no longer C3.PIN_PLUS, Q3.E
- net SUPPLY_UART_TX: now also U10.PB0, U8.PB0; no longer U7.PB0, U9.PB0
Other:
- moved on the sheet: C2, C3, C5, C7, C8, R10, R11, R15, R16, R17, R18, R19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

Commit message: I finished supply control schematics
Parts:
- added C10, C11: 10 uF, my_devices:C
- added C9: 1000 uF, my_devices:C
- added D9: D, my_devices:D
- added R26: 620, my_devices:R
- added R27: 1M, my_devices:R
- added R28, R29: 2M, my_devices:R
- added U14: 2004A I2C, my_devices:I2C_DISPLAY
- BAT3: value 6V ... 12V -> 10V ... 12V
- C2, C8: value 1000 uF -> 10 uF
- C5: value 0.1 uF -> 10 uF; device my_devices:C-1 -> my_devices:C
- C7: value 1000 uF -> 0.1 uF; device my_devices:C -> my_devices:C-1
- FU1, FU2: value H520PT / 0.5A -> H520PT / 1A
- R11, R6: value 10K -> 2M
- R12: value 1M -> 2M
- R13, R19: value 1M -> 10K
- R15: value 620 -> 1M
- R16: value 10K -> 1M
- R17: value 10K -> 620
- R18: value 620 -> 10K
- R20: value 2M -> 620
- R21: value 2M -> 1M
- R23: value GL5528 -> 2M; device my_devices:RF -> my_devices:R
- R24: value 620 -> 2M
- R25: value 1M -> GL5528; device my_devices:R -> my_devices:RF
- R7: value 3K -> 1M
- R8: value 2M -> 10K
- R9: value 2M -> 3K
- U10: value ATMEGA328P -> FAN73611; device my_devices:ATMEGA328P -> my_devices:FAN73611
- U11: value E220-900T22D -> ATMEGA328P; device my_devices:LORA -> my_devices:ATMEGA328P
- U12: value BME280BME280-CONNECTOR-ONLY -> E220-900T22D; device my_devices:BME280BME280-CONNECTOR-ONLY -> my_devices:LORA
- U13: value 2004A I2C -> BME280BME280-CONNECTOR-ONLY; device my_devices:I2C_DISPLAY -> my_devices:BME280BME280-CONNECTOR-ONLY
- U7: value FAN73611 -> MCP1703T-3302E/CB; device my_devices:FAN73611 -> my_devices:VOLTAGE_REGULATOR
- U8: value ATTINY13 -> FAN73611; device my_devices:ATTINY13 -> my_devices:FAN73611
- U9: value FAN73611 -> ATTINY13; device my_devices:FAN73611 -> my_devices:ATTINY13
Connections:
- new net N$2: D6.P$2, R6.P$2, R7.P$2, U2.D-
- new net N$28: D9.P$2, R28.P$2
- new net SUPPLY_CONTROL_3V3: C4.PIN_PLUS, U2.A-, U2.B-, U2.C-, U7.OUT
- net +12V: now also U10.VB, U10.VDD; no longer U9.VB, U9.VDD
- net +5V: now also C8.PIN_PLUS, R18.P$1, R19.P$2, R21.P$1, R23.P$2, R24.P$2, U11.AREF, U11.AVCC, U14.VCC; no longer C7.PIN_PLUS, R16.P$1, R17.P$2, R19.P$1, R20.P$2, R21.P$2, U10.AREF, U10.AVCC, U10.VCC
- net CURRENT_SUPPLY_IN_USE: now also R17.P$2, U9.PB1; no longer R15.P$2, U8.PB1
- net ENABLE_DISPLAY: now also R20.P$1, U11.PC3; no longer R18.P$1, U10.PC3
- net ENABLE_DR\YER: now also U10.IN, U11.PB1; no longer U10.PB1, U9.IN
- net FLOODING_ALARM_INDOOR: now also R24.P$1, U11.PC0; no longer R22.P$1, U10.PC0
- net FLOODING_ALARM_OUTDOOR: now also R22.P$1, U11.PC1; no longer R20.P$1, U10.PC1
- net GND: now also C10.PIN_GND, C11.PIN_GND, C5.PIN_GND, C7.P$2, C9.PIN_GND, R15.P$1, R16.P$1, R25.P$2, R27.P$1, R29.P$2, R7.P$1, U10.VS, U11.GND1, U13.GND, U8.VS; no longer C5.P$2, C7.PIN_GND, R11.P$1, R12.P$1, R23.P$2, R25.P$1, U10.GND1, U7.VS, U9.VS
- net I2C_SCL: now also U11.PC4, U14.SCL; no longer U10.PC4, U12.SCL
- net I2C_SDA: now also U11.PC5, U14.SDA; no longer U10.PC5, U12.SDA
- net IS_ENABLE_RESERVE_+5V_INV: now also U8.IN; no longer U7.IN
- net IS_PRIMARY_BATTERY_OK: now also D6.P$1; no longer U2.D-
- net IS_RESERVE_BATTERY_OK: now also D9.P$1; no longer D6.P$1
- net LIGHT_SENSOR: now also R21.P$2, R25.P$1, U11.PC2; no longer R19.P$2, R23.P$1, U10.PC2
- net LORA_AUX: now also U11.PD6, U12.AUX; no longer U10.PD6, U11.AUX
- net LORA_M0M1: now also U11.PD7, U12.M0, U12.M1; no longer U10.PD7, U11.M0, U11.M1
- net LORA_RX: now also U11.PD4, U12.RX; no longer U10.PD4, U11.RX
- net LORA_TX: now also U11.PD3, U12.TX; no longer U10.PD3, U11.TX
- net N$1: now also C10.PIN_PLUS
- net N$10: now also U14.GND; no longer U13.GND
- net N$11: now also R20.P$2; no longer R18.P$2
- net N$16: now also R18.P$2, U11.PD2; no longer R16.P$2, U10.PD2
- net N$17: now also U9.PB5; no longer U8.PB5
- net N$23: now also C9.PIN_PLUS, R26.P$1, R27.P$2; no longer C8.PIN_PLUS, R24.P$1, R25.P$2
- net N$24: now also R26.P$2; no longer R24.P$2
- net N$25: now also R8.P$1; no longer R6.P$1
- net N$27: now also R9.P$1; no longer R7.P$1
- net N$29: now also C5.PIN_PLUS, R13.P$2, R17.P$1, R8.P$2, R9.P$2; no longer C4.PIN_PLUS, R11.P$2, R15.P$1, R6.P$2, R7.P$2
- net N$5: now also C11.PIN_PLUS
- net N$6: now also U10.HO; no longer U9.HO
- net N$7: now also C7.P$1, R19.P$1, U11.PC6; no longer C6.P$1, R17.P$1, U10.PC6
- net N$9: now also R28.P$1, R29.P$1; no longer D6.P$2
- net OPEN_DOOR_ALARM: now also R23.P$1, U11.PB3; no longer R21.P$1, U10.PB3
- net PRIMARY_SUPPLY_12V: now also R11.P$2; no longer R9.P$2
- net PRIMARY_VOLTAGE_LEVEL: now also R11.P$1, R15.P$2, U9.PB3; no longer R13.P$2, R9.P$1, U8.PB3
- net REQUEST_SUPPLY_MEASURE_INV: now also U11.PB2; no longer U10.PB2
- net RESERVE_+5V_LEVEL: now also R10.P$1, R14.P$2, U9.PB2; no longer R12.P$2, R8.P$1, U8.PB2
- net RESERVE_+5V_SUPPLY: now also R10.P$2, U8.VB, U8.VDD; no longer R8.P$2, U7.VB, U7.VDD
- net RESERVE_SUPPLY_12V: now also R12.P$2; no longer R10.P$2
- net RESERVE_VOLTAGE_LEVEL: now also R12.P$1, R16.P$2, U9.PB4; no longer R10.P$1, R14.P$2, U8.PB4
- net SUPPLY_AVR_+5V: now also C6.P$1, U9.VCC; no longer C5.P$1, U8.VCC
- net SUPPLY_CONTROL_+5V: now also R6.P$1, U7.IN; no longer U2.A-, U2.B-, U2.C-
- net SUPPLY_UART_TX: now also U11.PB0, U9.PB0; no longer U10.PB0, U8.PB0
- net USE_RESERVE_5V_BATTERY: now also U8.HO; no longer U7.HO
Other:
- note added: "WARNING If you want to change nominals - you must check voltage at legs D+ and D- in 4 cases. My measuremets showed in [brackeds] for example Case #1 (PRIM OK, RESERVE OK): D+ < D- [2.4V < 4.8V] Case #2 (PRIM OK RESERVE BAD): D+ < D- [0V < 4.8V] Case #3 (PRIM BAD, RESERVE OK): D+ > D- [2.4V > 1.6V] Case #4 (PRIM BAD, RESERVE BAD, SUPPLY_CONTROL_+5V line OK): D+ < D- [0V < 1.6V]"
- moved on the sheet: BAT1, BAT2, BAT3, C1, C2, C3, C4, C6, C8, D1, D2, D3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
